Commit message: .

File: ros2_new_ws/src/my_robot_description/urdf/common_properties.urdf.xacro (robot description, xacro)
@@ -6,4 +6,7 @@
     <material name = "grey">
         <color rgba = "0.5 0.5 0.5 1"></color>
+    </material>
+    <material name = "red">
+        <color rgba = "1 0 0 1"></color>
     </material>
     <xacro:macro name="box_inertia" params="m l w h xyz rpy">

File: ros2_new_ws/src/my_robot_description/urdf/mobile_base_gazebo.xacro (robot description, xacro)
@@ -36,3 +36,23 @@
         </plugin>
     </gazebo>
+    <gazebo>
+        <plugin name="diff_front_drive_controller" filename="libgazebo_ros_diff_drive.so">
+            <!-- Update rate in Hz -->
+            <update_rate>50</update_rate>
+            <!-- wheels -->
+            <left_joint>base_left_front_wheel_joint</left_joint>
+            <right_joint>base_right_front_wheel_joint</right_joint>
+            <!-- kinematics -->
+            <wheel_separation>0.45</wheel_separation> <!--it is the distance between the center of two wheels,
+            which is "base_width + wheel_length" ).4 + 0.05-->
+            <wheel_diameter>0.2</wheel_diameter>
+            <!-- output -->
+            <publish_odom>true</publish_odom> <!-- where the robot is compared to the origin-->
+            <publish_odom_tf>true</publish_odom_tf>
+            <publish_wheel_tf>true</publish_wheel_tf>
+            <odometry_topic>odom</odometry_topic>
+            <odometry_frame>odom</odometry_frame>
+            <robot_base_frame>base_footprint_link</robot_base_frame>
+        </plugin>
+    </gazebo>
 </robot>

File: ros2_new_ws/src/my_robot_description/urdf/my_robot.urdf.xacro (robot description, xacro)
@@ -4,3 +4,4 @@
     <xacro:include filename="mobile_base.urdf.xacro" />
     <xacro:include filename="mobile_base_gazebo.xacro" />
+    <xacro:include filename="lidar.xacro" />
 </robot>

Commit message: '.'

File: ros2_new_ws/src/my_robot_description/urdf/common_properties.urdf.xacro (robot description, xacro)
@@ -9,4 +9,7 @@
     <material name = "red">
         <color rgba = "1 0 0 1"></color>
+    </material>
+    <material name = "green">
+        <color rgba = "0 1 0 1"></color>
     </material>
     <xacro:macro name="box_inertia" params="m l w h xyz rpy">

File: ros2_new_ws/src/my_robot_description/urdf/lidar.xacro (robot description, xacro)
@@ -49,5 +49,7 @@
             </ray>
             <plugin name="lidar_controller" filename="libgazebo_ros_ray_sensor.so">
-                <topicName>/scan</topicName>
+                <ros>
+                    <argument>~/out:=scan</argument>
+                </ros>
                 <output_type>sensor_msgs/LaserScan</output_type>
                 <frame_name>lidar_link</frame_name>
@@ -56,2 +58,40 @@
     </gazebo>
 </robot>
+<gazebo reference="ultrasonic_link">
+        <material>Gazebo/Green</material>
+        <sensor type="ray" name="ultrasonic_link">
+        <pose>0 0 0 0 0 0</pose>
+        <visualize>true</visualize>
+        <update_rate>20</update_rate>
+        <ray>
+            <scan>
+                <horizontal>
+                <samples>1</samples>
+                <resolution>1</resolution>
+                <min_angle>0</min_angle>
+                <max_angle>0</max_angle>
+                </horizontal>
+                <vertical>
+                <samples>1</samples>
+                <resolution>1</resolution>
+                <min_angle>0</min_angle>
+                <max_angle>0</max_angle>
+                </vertical>
+            </scan>
+            <range>
+                <min>0.02</min>
+                <max>4.0</max>
+                <resolution>0.01</resolution>
+            </range>
+        </ray>
+        <plugin filename="libgazebo_ros_range.so" name="gazebo_ros_range">
+            <!-- <gaussianNoise>0.01</gaussianNoise> -->
+            <alwaysOn>true</alwaysOn>
+            <updateRate>20</updateRate>
+            <topicName>sensor/ultrasonic</topicName>
+            <frameName>ultrasonic_link</frameName>
+            <radiation>SOUND</radiation>
+            <fov>0.1</fov>
+        </plugin>
+        </sensor>
+    </gazebo>

File: ros2_new_ws/src/my_robot_description/urdf/my_robot.urdf.xacro (robot description, xacro)
@@ -4,4 +4,5 @@
     <xacro:include filename="mobile_base.urdf.xacro" />
     <xacro:include filename="mobile_base_gazebo.xacro" />
-    <xacro:include filename="lidar.xacro" />
+    <!-- <xacro:include filename="lidar.xacro" /> -->
+    <xacro:include filename="ultrasonic.xacro" />
 </robot>
