Commit message: /

File: ros2_new_ws/src/my_robot_description/urdf/lidar.xacro (robot description, xacro)
@@ -58,40 +58,2 @@
     </gazebo>
 </robot>
-<gazebo reference="ultrasonic_link">
-        <material>Gazebo/Green</material>
-        <sensor type="ray" name="ultrasonic_link">
-        <pose>0 0 0 0 0 0</pose>
-        <visualize>true</visualize>
-        <update_rate>20</update_rate>
-        <ray>
-            <scan>
-                <horizontal>
-                <samples>1</samples>
-                <resolution>1</resolution>
-                <min_angle>0</min_angle>
-                <max_angle>0</max_angle>
-                </horizontal>
-                <vertical>
-                <samples>1</samples>
-                <resolution>1</resolution>
-                <min_angle>0</min_angle>
-                <max_angle>0</max_angle>
-                </vertical>
-            </scan>
-            <range>
-                <min>0.02</min>
-                <max>4.0</max>
-                <resolution>0.01</resolution>
-            </range>
-        </ray>
-        <plugin filename="libgazebo_ros_range.so" name="gazebo_ros_range">
-            <!-- <gaussianNoise>0.01</gaussianNoise> -->
-            <alwaysOn>true</alwaysOn>
-            <updateRate>20</updateRate>
-            <topicName>sensor/ultrasonic</topicName>
-            <frameName>ultrasonic_link</frameName>
-            <radiation>SOUND</radiation>
-            <fov>0.1</fov>
-        </plugin>
-        </sensor>
-    </gazebo>

File: ros2_new_ws/src/my_robot_description/urdf/ultrasonic.xacro (robot description, xacro)
@@ -25,28 +25,30 @@
     </joint>
     <gazebo reference="ultrasonic_link">
-        <material>Gazebo/Green</material>
-        <sensor type="gpu_ray" name="range_sensor">
+        <material>Gazebo/Red</material>
+        <sensor name="ultrasonic" type="ray">
+            <pose>0 0 0 0 0 0</pose>
+            <always_on>true</always_on>
             <visualize>true</visualize>
+            <update_rate>10</update_rate>
             <ray>
                 <scan>
                     <horizontal>
-                        <samples>10</samples>
-                        <resolution>1</resolution>
-                        <min_angle>-0.087</min_angle>
-                        <max_angle>0.087</max_angle>
+                        <samples>5</samples>
+                        <resolution>1.000000</resolution>
+                        <min_angle>-0.12</min_angle>
+                        <max_angle>0.12</max_angle>
                     </horizontal>
                     <vertical>
-                        <samples>10</samples>
-                        <resolution>1</resolution>
-                        <min_angle>-0.087</min_angle>
-                        <max_angle>0.087</max_angle>
+                        <samples>5</samples>
+                        <resolution>1.000000</resolution>
+                        <min_angle>-0.01</min_angle>
+                        <max_angle>0.01</max_angle>
                     </vertical>
                 </scan>
                 <range>
-                    <min>0.10</min>
-                    <max>5.0</max>
-                    <resolution>1</resolution>
+                    <min>0.02</min>
+                    <max>4</max>
+                    <resolution>0.01</resolution>
                 </range>
-            <!-- Using gazebo's noise instead of plugin's -->
                 <noise>
                     <type>gaussian</type>
@@ -55,17 +57,13 @@
                 </noise>
             </ray>
-            <!-- Using gazebo's update rate instead of plugin's -->
-            <update_rate>30</update_rate>
-            <plugin name="ultrasonic_controller" filename="libgazebo_ros_ray_sensor.so">
-            <!-- Change namespace and output topic so published topic is /rrbot/laser/scan -->
+            <plugin name="ultrasonic" filename="libgazebo_ros_ray_sensor.so">
                 <ros>
-                    <!-- <namespace>/rrbot</namespace> -->
                     <remapping>~/out:=range</remapping>
                 </ros>
-            <!-- Set output to sensor_msgs/Range to get same output type as gazebo_ros_range -->
                 <output_type>sensor_msgs/Range</output_type>
+                <radiation_type>ultrasound</radiation_type>
                 <frame_name>ultrasonic_link</frame_name>
             </plugin>
         </sensor>
-    </gazebo>
+   </gazebo>
 </robot>
